File: CartridgeBreakout.kicad_pcb (KiCad board)
At the start: 2 copper layers, 99 x 75 mm, 23 parts, among them J1 Conn_02x10_Odd_Even, J10 Conn_01x02, J2 Conn_02x10_Odd_Even, J3 Conn_02x10_Odd_Even, J4 Conn_02x10_Odd_Even, J5 Conn_02x10_Odd_Even, J6 Conn_02x10_Odd_Even, J7 EXPANSION_PORT_C64_EDGE, J8 Conn_02x05_Odd_Even, J9 Conn_01x03

Commit message: Converted to KiCAD 6 format
Other:
- net class Default removed
- net class Power removed
